File: pcb_files/adalogger_shield_v1.brd (EAGLE design)
At the start: 50.8 x 22.9 mm, 5 parts

Commit message: bLayer is OK
Parts:
- moved UART 13.5 mm to (22.7, 11.4), turned to 90 degrees
- moved A/D 2.95 mm to (7.84, 11.4)
- moved I2C 0.35 mm to (42.9, 11.4)
Routing:
- net 3V: track 0.00 -> 74.5 mm
- net GND: track 0.00 -> 45.2 mm
- net TX: track 0.00 -> 22.7 mm
- net RX: track 0.00 -> 19.5 mm
- net A2: track 0.00 -> 17.2 mm
- net A1: track 0.00 -> 14.0 mm
- net SDA: track 0.00 -> 9.67 mm
- net SCL: track 0.00 -> 7.64 mm

Commit message: second version ready
Parts:
- moved UART 1.90 mm to (24.6, 11.4)
Routing:
- net 3V: track 74.5 -> 47.2 mm
- net GND: track 45.2 -> 50.4 mm
- net TX: track 22.7 -> 21.0 mm
- net RX: track 19.5 -> 18.3 mm

Commit message: design ok
Parts:
- moved UART 7.11 mm to (31.7, 11.4)
Routing:
- net RX: track 18.3 -> 10.9 mm
- net TX: track 21.0 -> 13.9 mm
- net GND: track 50.4 -> 45.3 mm
- net SDA: track 10.1 -> 11.4 mm
